Commit message: Working green object pick pack with gripper

File: pick_place_exercise/urdf/ur_robotiq85_macro.xacro (robot description, xacro)
@@ -2,11 +2,63 @@
 <robot xmlns:xacro="http://ros.org/wiki/xacro"
        name="ur5_robotiq85" >
-	<xacro:arg name="limited" default="true"/>
-	<!-- UR5e  -->
-	<xacro:include filename="$(find ur_description)/urdf/ur.urdf.xacro" />
+	<!-- Arguments -->
+	<xacro:arg name="ur_type" default="ur5e"/>
+	<xacro:arg name="tf_prefix" default="" />
+	<xacro:arg name="joint_limit_params" default="$(find ur_description)/config/$(arg ur_type)/joint_limits.yaml"/>
+	<xacro:arg name="kinematics_params" default="$(find ur_description)/config/$(arg ur_type)/default_kinematics.yaml"/>
+	<xacro:arg name="physical_params" default="$(find ur_description)/config/$(arg ur_type)/physical_parameters.yaml"/>
+	<xacro:arg name="visual_params" default="$(find ur_description)/config/$(arg ur_type)/visual_parameters.yaml"/>
+	<xacro:arg name="safety_limits" default="false"/>
+	<xacro:arg name="safety_pos_margin" default="0.15"/>
+	<xacro:arg name="safety_k_position" default="20"/>
+	<!-- ros2_control related parameters -->
+	<xacro:arg name="headless_mode" default="false" />
+	<xacro:arg name="robot_ip" default="0.0.0.0" />
+	<xacro:arg name="script_filename" default=""/>
+	<xacro:arg name="output_recipe_filename" default=""/>
+	<xacro:arg name="input_recipe_filename" default=""/>
+	<!-- Simulation parameters -->
+	<xacro:arg name="use_fake_hardware" default="false" />
+	<xacro:arg name="fake_sensor_commands" default="false" />
+	<xacro:arg name="sim_gazebo" default="false" />
+	<xacro:arg name="simulation_controllers" default="" />
+	<!-- Import UR macro -->
+	<xacro:include filename="$(find ur_description)/urdf/ur_macro.xacro"/>
+	<!-- Instantiate UR robot -->
+	<xacro:ur_robot
+		name="ur"
+		tf_prefix="$(arg tf_prefix)"
+		parent="world"
+		joint_limits_parameters_file="$(arg joint_limit_params)"
+		kinematics_parameters_file="$(arg kinematics_params)"
+		physical_parameters_file="$(arg physical_params)"
+		visual_parameters_file="$(arg visual_params)"
+		safety_limits="$(arg safety_limits)"
+		safety_pos_margin="$(arg safety_pos_margin)"
+		safety_k_position="$(arg safety_k_position)"
+		use_fake_hardware="$(arg use_fake_hardware)"
+		fake_sensor_commands="$(arg fake_sensor_commands)"
+		sim_gazebo="$(arg sim_gazebo)"
+		sim_ignition="false"
+		headless_mode="$(arg headless_mode)"
+		initial_positions="${dict(shoulder_pan_joint=0.0,shoulder_lift_joint=-1.57,elbow_joint=0.0,wrist_1_joint=-1.57,wrist_2_joint=0.0,wrist_3_joint=0.0)}"
+		script_filename="$(arg script_filename)"
+		output_recipe_filename="$(arg output_recipe_filename)"
+		input_recipe_filename="$(arg input_recipe_filename)"
+		robot_ip="$(arg robot_ip)">
+		<origin xyz="0 0 0" rpy="0 0 0" />
+	</xacro:ur_robot>
 	<!-- Robotiq 85 -->
 	<xacro:include filename="$(find robotiq_description)/urdf/robotiq_2f_85_macro.urdf.xacro" />
-	<xacro:robotiq_gripper prefix="" parent="flange">
+	<xacro:robotiq_gripper prefix="" parent="tool0">
 		<origin xyz="0 0 0" rpy="0 0 0" />
 	</xacro:robotiq_gripper>
+	<!-- Gazebo ros2_control plugin -->
+	<xacro:if value="$(arg sim_gazebo)">
+		<gazebo>
+			<plugin filename="libgazebo_ros2_control.so" name="gazebo_ros2_control">
+				<parameters>$(arg simulation_controllers)</parameters>
+			</plugin>
+		</gazebo>
+	</xacro:if>
 </robot>

File: pick_place_exercise/urdf/ur_robotiq85_test.xacro (robot description, xacro)
@@ -2,6 +2,58 @@
 <robot xmlns:xacro="http://ros.org/wiki/xacro"
        name="ur5_robotiq85" >
-	<xacro:arg name="limited" default="true"/>
-	<!-- UR5e  -->
-	<xacro:include filename="$(find ur_description)/urdf/ur.urdf.xacro" />
+	<!-- Arguments -->
+	<xacro:arg name="ur_type" default="ur5e"/>
+	<xacro:arg name="tf_prefix" default="" />
+	<xacro:arg name="joint_limit_params" default="$(find ur_description)/config/$(arg ur_type)/joint_limits.yaml"/>
+	<xacro:arg name="kinematics_params" default="$(find ur_description)/config/$(arg ur_type)/default_kinematics.yaml"/>
+	<xacro:arg name="physical_params" default="$(find ur_description)/config/$(arg ur_type)/physical_parameters.yaml"/>
+	<xacro:arg name="visual_params" default="$(find ur_description)/config/$(arg ur_type)/visual_parameters.yaml"/>
+	<xacro:arg name="safety_limits" default="false"/>
+	<xacro:arg name="safety_pos_margin" default="0.15"/>
+	<xacro:arg name="safety_k_position" default="20"/>
+	<!-- ros2_control related parameters -->
+	<xacro:arg name="headless_mode" default="false" />
+	<xacro:arg name="robot_ip" default="0.0.0.0" />
+	<xacro:arg name="script_filename" default=""/>
+	<xacro:arg name="output_recipe_filename" default=""/>
+	<xacro:arg name="input_recipe_filename" default=""/>
+	<!-- Simulation parameters -->
+	<xacro:arg name="use_fake_hardware" default="false" />
+	<xacro:arg name="fake_sensor_commands" default="false" />
+	<xacro:arg name="sim_gazebo" default="false" />
+	<xacro:arg name="simulation_controllers" default="" />
+	<!-- Import UR macro -->
+	<xacro:include filename="$(find ur_description)/urdf/ur_macro.xacro"/>
+	<!-- Instantiate UR robot -->
+	<xacro:ur_robot
+		name="ur"
+		tf_prefix="$(arg tf_prefix)"
+		parent="world"
+		joint_limits_parameters_file="$(arg joint_limit_params)"
+		kinematics_parameters_file="$(arg kinematics_params)"
+		physical_parameters_file="$(arg physical_params)"
+		visual_parameters_file="$(arg visual_params)"
+		safety_limits="$(arg safety_limits)"
+		safety_pos_margin="$(arg safety_pos_margin)"
+		safety_k_position="$(arg safety_k_position)"
+		use_fake_hardware="$(arg use_fake_hardware)"
+		fake_sensor_commands="$(arg fake_sensor_commands)"
+		sim_gazebo="$(arg sim_gazebo)"
+		sim_ignition="false"
+		headless_mode="$(arg headless_mode)"
+		initial_positions="${dict(shoulder_pan_joint=0.0,shoulder_lift_joint=-1.57,elbow_joint=0.0,wrist_1_joint=-1.57,wrist_2_joint=0.0,wrist_3_joint=0.0)}"
+		script_filename="$(arg script_filename)"
+		output_recipe_filename="$(arg output_recipe_filename)"
+		input_recipe_filename="$(arg input_recipe_filename)"
+		robot_ip="$(arg robot_ip)">
+		<origin xyz="0 0 0" rpy="0 0 0" />
+	</xacro:ur_robot>
+	<!-- Gazebo ros2_control plugin -->
+	<xacro:if value="$(arg sim_gazebo)">
+		<gazebo>
+			<plugin filename="libgazebo_ros2_control.so" name="gazebo_ros2_control">
+				<parameters>$(arg simulation_controllers)</parameters>
+			</plugin>
+		</gazebo>
+	</xacro:if>
 </robot>
